Commit message: upgraded structure

File: description/lance.urdf (robot description, URDF)
Before this commit: robot None, 6 links, 5 joints
Links:
- link collection_link: geometry collision mesh filename=file://$(find lance_sim)/description/lance/meshes/lance-202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; visual mesh filename=file://$(find lance_sim)/description/lance/meshes/lance-202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
- link frame_link: geometry collision mesh filename=file://$(find lance_sim)/description/lance/meshes/lance-202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; visual mesh filename=file://$(find lance_sim)/description/lance/meshes/lance-202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
- link left_track_link: geometry collision mesh filename=file://$(find lance_sim)/description/lance/meshes/lance-202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; visual mesh filename=file://$(find lance_sim)/description/lance/meshes/lance-202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
- link lidar_link: geometry collision cylinder length=0.098 radius=0.048; visual mesh filename=file://$(find lance_sim)/description/lance/meshes/lance-202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
- link right_track_link: geometry collision mesh filename=file://$(find lance_sim)/description/lance/meshes/lance-202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; visual mesh filename=file://$(find lance_sim)/description/lance/meshes/lance-202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
