Commit message: debug and camera tfs

File: lance_sim/description/lance.urdf (robot description, URDF)
Before this commit: robot lance, 6 links, 5 joints
Links:
- added link fwd_cam_link
Joints:
- added joint fwd_cam_joint: type fixed, parent frame_link, child fwd_cam_link, origin xyz=0.72468246 0 0.51148737 rpy=-1.74532925199 0 -1.57079632679

Commit message: huh

File: lance_sim/description/lance.urdf (robot description, URDF)
Before this commit: robot lance, 7 links, 6 joints
Links:
- added link left_cam_link
- added link rght_cam_link
Joints:
- added joint left_cam_joint: type fixed, parent frame_link, child left_cam_link, origin xyz=-0.06416965 0.28448800 0.22203322 rpy=-1.57079632679 0 0
- added joint rght_cam_joint: type fixed, parent frame_link, child rght_cam_link, origin xyz=-0.06416965 -0.28448800 0.22203322 rpy=-1.57079632679 0 3.1415926
